File: psion.sch (EAGLE design)
At the start: 92 parts, among them J2 1-2295018-2, Q1 NTF3055L108T1G, Q2 MMBT2907ALT1G, Q3 NTF3055L108T1G, Q5 MOSFET-PCH_SOT-223, Q6 MOSFET-PCH_SOT-223, T1 2908-05WB-MG, U2 HV823LG-G, U3 ATMEGA32U4-AU, U4 OSD3358-512M-BCB, U5 MAX1620EEE+, U6 MAX1620EEE+, U7 ATTINY404-SSN, U8 TPS61090RSAR, Y1 ABM10-16.000MHZ-D30-T3

Commit message: work on lcd bias power + pdfs
Parts:
- removed C13, C6, C7: 22uf, gothack:CPOL-USKEMET_C_2312
- removed C3, C4: 0.1uf, dp_devices:CAPACITOR_NPOL-0805
- removed C5: 100pf, dp_devices:CAPACITOR_NPOL-0805
- removed D2, D3, D6: MBRS0540, ipc-7351-diode:SCHOTTKY_SOD-123
- removed L1: LQH2MCN270K02L, microbuilder:INDUCTOR
- removed Q1: NTF3055L108T1G, SparkFun-DiscreteSemi:MOSFET-NCHANNELSMD
- removed R5: 1M, resistor:R-EU_R0805
- removed R6: 300k, resistor:R-EU_R0805
- removed R7: 3.3M, resistor:R-EU_R0805
- removed R8: 2.2M, resistor:R-EU_R0805
- added C25, C26: 0.1uf, dp_devices:CAPACITOR_NPOL-0805
- added C27, C30: 100pf, dp_devices:CAPACITOR_NPOL-0805
- added C28, C29: 22uf, gothack:CPOL-USKEMET_C_2312
- added D10, D11, D9: MBRS0540, ipc-7351-diode:SCHOTTKY_SOD-123
- added L5: LQH2MCN270K02L, microbuilder:INDUCTOR
- added Q8: MMBT2907ALT1G, ipc-7351-transistor:PNP_SOT-23
- added R27: 2.2M, resistor:R-EU_R0805
- added R28, R30: 10k, resistor:R-EU_R0805
- added R29: 3.3M, resistor:R-EU_R0805
- C10: value 22uf -> 100pf; device gothack:CPOL-USKEMET_C_2312 -> dp_devices:CAPACITOR_NPOL-0805
- C11: value 1uf -> 22uf; device dp_devices:CAPACITOR_NPOL-0805 -> gothack:CPOL-USKEMET_C_2312
- C12: value 100pf -> 22uf; device dp_devices:CAPACITOR_NPOL-0805 -> gothack:CPOL-USKEMET_C_2312
- Q2: value MMBT2907ALT1G -> NTF3055L108T1G; device ipc-7351-transistor:PNP_SOT-23 -> SparkFun-DiscreteSemi:MOSFET-NCHANNELSMD
- R10: value 931k -> 300k
- R11: value 300k -> 1M
- R12: value 2.94M -> 300k
- R13: value 10k -> 3.3M
- R14: value 10k -> 2.2M
- R9: value 2.2M -> 1M
Connections:
- removed net N$18: Q1.G, U5.DHI, U5.DLO
- removed net N$19: D2.A, L1.2, Q1.D, U5.LX
- removed net N$20: R5.1, U5.DOUT
- removed net N$21: C5.1, R5.2, R6.1, R7.2, U5.FB
- removed net N$22: C5.2, C7.+, D2.K, Q2.E, R7.1, R8.1
- removed net N$30: D5.K, R13.1, U5.BATT
- removed net N$31: C4.1, D5.A, U5.REF
- new net N$45: D5.K, R28.1, U5.BATT
- new net N$46: C9.1, D5.A, U5.REF
- new net N$47: R9.1, U6.DOUT
- new net N$48: C27.1, R10.1, R29.2, R9.2, U6.FB
- new net N$49: D10.K, R30.1, U6.BATT
- new net N$50: C26.1, D10.A, U6.REF
- new net N$51: C30.2, D11.A, D9.K
- net +3V3: now also C25.1; no longer C3.1
- net GND: now also C11.-, C12.-, C25.2, C26.2, C28.-, C29.+, Q2.S, R10.2, R12.2; no longer C10.-, C13.-, C3.2, C4.2, C6.-, C7.-, Q1.S, R6.2
- net LCD_BIAS_N: now also C27.2, C29.-, D9.A, R29.1; no longer C12.2, C13.+, D3.A, R12.1
- net LCD_BIAS_P: now also Q8.C; no longer Q2.C
- net N$16: now also U5.DHI, U5.DLO; no longer U6.DHI, U6.DLO
- net N$17: now also D4.A, U5.LX; no longer C11.1, U6.LX
- net N$23: now also Q2.G, U6.DHI, U6.DLO; no longer Q2.B, R8.2, R9.1
- net N$24: now also C30.1, L5.2, Q2.D, U6.LX; no longer R9.2, U5.LCDON_
- net N$25: now also R11.1, U5.DOUT; no longer R10.1, U6.DOUT
- net N$26: now also C10.1, R11.2, R12.1, R13.2, U5.FB; no longer C12.1, R10.2, R11.1, R12.2, U6.FB
- net N$27: now also C10.2, C12.+, D4.K, Q8.E, R13.1; no longer D6.K, U6.BATT
- net N$28: now also Q8.B, R14.2, R27.1; no longer C9.1, D6.A, R11.2, U6.REF
- net N$32: now also R27.2, U5.LCDON_; no longer C11.2, D3.K, D4.A
- net VCCINT: now also C11.+, C28.+, D11.K, L5.1, R28.2, R30.2; no longer C10.+, C6.+, D4.K, L1.1, R13.2, R14.2
Other:
- moved on the sheet: C8, C9, D4, D5, L2, Q3, R10, R11, R12, R13, R14, R9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

Commit message: routing + gerbers + pdfs + docs
Connections:
- net N$15 renamed EL_VA_PRE
- net N$17 renamed LCD_BIAS_P_P1
- net N$24 renamed LCD_BIAS_N_P1
- net N$27 renamed LCD_BIAS_P_P2
- net N$36 renamed USBC_IND_SW
- net N$41 renamed USBC_VBUS_SW
- net N$51 renamed LCD_BIAS_N_P2
- net LCD_BIASN_DN: now also U7.PA5; no longer U7.PA6
- net LCD_BIASN_SHDN_: now also U7.PA7; no longer U7.PA5
- net LCD_BIASN_UP: now also U7.PA6; no longer U7.PA7
- net LCD_BIASP_SHDN_: now also U7.PA3; no longer U7.PA1
- net LCD_BIASP_UP: now also U7.PA1; no longer U7.PA3
Other:
- moved on the sheet: R4
Changed lines of the file:
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@@
 <setting verticaltext="up"/>
 </settings>
-<grid distance="0.1" unitdist="inch" unit="inch" style="lines" multiple="1" display="no" altdistance="0.01" altunitdist="inch" altunit="inch"/>
+<grid distance="0.1" unitdist="inch" unit="mil" style="lines" multiple="1" display="no" altdistance="50" altunitdist="mil" altunit="mil"/>
 <layers>
 <layer number="1" name="Top" color="4" fill="1" visible="no" active="no"/>
@@
 </class>
 <class number="1" name="data" width="0.1524" drill="0.2794">
-<clearance class="0" value="0.1778"/>
 <clearance class="1" value="0.0889"/>
 </class>
 <class number="2" name="power" width="0.254" drill="0.2794">
-<clearance class="0" value="0.1524"/>
-<clearance class="1" value="0.1524"/>
 <clearance class="2" value="0.1524"/>
 </class>
 <class number="3" name="data_usb" width="0.1524" drill="0.2794">
-<clearance class="0" value="0.1778"/>
-<clearance class="1" value="0.1778"/>
-<clearance class="2" value="0.1778"/>
 <clearance class="3" value="0.0889"/>
 </class>
 <class number="4" name="data_lcd" width="0.1524" drill="0.2794">
-<clearance class="0" value="0.1778"/>
-<clearance class="1" value="0.1778"/>
-<clearance class="2" value="0.1778"/>
-<clearance class="3" value="0.1778"/>
 <clearance class="4" value="0.0889"/>
 </class>
 <class number="5" name="data_lowspeed" width="0.1524" drill="0.2794">
-<clearance class="0" value="0.1778"/>
-<clearance class="1" value="0.1778"/>
-<clearance class="2" value="0.1778"/>
-<clearance class="3" value="0.1778"/>
-<clearance class="4" value="0.1778"/>
 <clearance class="5" value="0.0889"/>
 </class>
@@
 </segment>
 </net>
-<net name="VIN_AC" class="0">
+<net name="VIN_AC" class="2">
 <segment>
 <pinref part="U4" gate="A" pin="VIN_AC@1"/>
@@
 </segment>
 </net>
-<net name="VIN_USB" class="0">
+<net name="VIN_USB" class="2">
 <segment>
 <pinref part="U4" gate="A" pin="VIN_USB@1"/>
@@
 </segment>
 </net>
-<net name="IOD_VCC33" class="0">
+<net name="IOD_VCC33" class="2">
 <segment>
 <pinref part="U4" gate="A" pin="SYS_VDD3_3P3V@1"/>
@@
 </segment>
 </net>
-<net name="SYS_RTC_1P8V" class="0">
+<net name="SYS_RTC_1P8V" class="2">
 <segment>
 <pinref part="U4" gate="A" pin="SYS_RTC_1P8V@4"/>
@@
 </segment>
 </net>
-<net name="VCC18" class="0">
+<net name="VCC18" class="2">
 <segment>
 <pinref part="U4" gate="A" pin="SYS_VDD_1P8V@10"/>
@@
 </segment>
 </net>
-<net name="N$36" class="0">
+<net name="USBC_IND_SW" class="2">
 <segment>
 <pinref part="U8" gate="G$1" pin="SW"/>
@@
 </segment>
 </net>
-<net name="N$41" class="0">
+<net name="USBC_VBUS_SW" class="2">
 <segment>
 <pinref part="Q5" gate="G$1" pin="S"/>
@@
 <attribute name="VALUE" x="231.14" y="72.2" size="2.0828" layer="96" ratio="10" rot="SR0"/>
 </instance>
-<instance part="R4" gate="G$1" x="220.98" y="91.44" smashed="yes">
-<attribute name="NAME" x="217.17" y="92.9386" size="1.778" layer="95"/>
-<attribute name="VALUE" x="217.17" y="88.138" size="1.778" layer="96"/>
+<instance part="R4" gate="G$1" x="218.44" y="91.44" smashed="yes">
+<attribute name="NAME" x="214.63" y="92.9386" size="1.778" layer="95"/>
+<attribute name="VALUE" x="214.63" y="88.138" size="1.778" layer="96"/>
 </instance>
 <instance part="U7" gate="G$1" x="218.44" y="27.94" smashed="yes">
@@
 </instance>
 <instance part="L2" gate="G$1" x="119.38" y="137.16" smashed="yes">
-<attribute name="NAME" x="115.57" y="140.97" size="1.778" layer="95"/>
-<attribute name="VALUE" x="115.57" y="134.62" size="1.778" layer="96"/>
+<attribute name="NAME" x="115.57" y="139.7" size="1.778" layer="95"/>
+<attribute name="VALUE" x="115.57" y="142.24" size="1.778" layer="96"/>
 </instance>
 <instance part="D4" gate="G$1" x="137.16" y="137.16" smashed="yes">
@@
 <instance part="D5" gate="G$1" x="76.2" y="124.46" smashed="yes" rot="R90">
 <attribute name="NAME" x="74.295" y="121.92" size="1.778" layer="95" rot="R90"/>
-<attribute name="VALUE" x="80.01" y="121.92" size="1.778" layer="96" rot="R90"/>
+<attribute name="VALUE" x="72.39" y="121.92" size="1.778" layer="96" rot="R90"/>
 </instance>
 <instance part="R28" gate="G$1" x="81.28" y="132.08" smashed="yes" rot="R90">
@@
 <bus name="LCD_EL:EL_VA,EL_VB,GND">
 <segment>
-<wire x1="220.98" y1="83.82" x2="215.9" y2="83.82" width="0.762" layer="92"/>
-<label x="215.9" y="81.28" size="1.778" layer="95" rot="MR180"/>
+<wire x1="218.44" y1="83.82" x2="213.36" y2="83.82" width="0.762" layer="92"/>
+<label x="218.44" y="81.28" size="1.778" layer="95" rot="MR180"/>
 </segment>
 <segment>
@@
 </segment>
 </net>
-<net name="KBDAVR_VCC" class="0">
+<net name="KBDAVR_VCC" class="2">
 <segment>
 <pinref part="U3" gate="A" pin="AVCC"/>
@@
 </segment>
 </net>
-<net name="EL_VB" class="0">
+<net name="EL_VB" class="2">
 <segment>
 <pinref part="U2" gate="G$1" pin="VB"/>
-<wire x1="226.06" y1="86.36" x2="218.44" y2="86.36" width="0.1524" layer="91"/>
-<wire x1="218.44" y1="86.36" x2="218.44" y2="83.82" width="0.1524" layer="91"/>
+<wire x1="226.06" y1="86.36" x2="215.9" y2="86.36" width="0.1524" layer="91"/>
+<wire x1="215.9" y1="86.36" x2="215.9" y2="83.82" width="0.1524" layer="91"/>
 </segment>
 <segment>
@@
 </segment>
 </net>
-<net name="N$15" class="0">
+<net name="EL_VA_PRE" class="2">
 <segment>
 <pinref part="U2" gate="G$1" pin="VA"/>
 <pinref part="R4" gate="G$1" pin="2"/>
+<wire x1="223.52" y1="91.44" x2="226.06" y2="91.44" width="0.1524" layer="91"/>
 </segment>
 </net>
-<net name="EL_VA" class="0">
+<net name="EL_VA" class="2">
 <segment>
 <pinref part="R4" gate="G$1" pin="1"/>
-<wire x1="215.9" y1="91.44" x2="215.9" y2="83.82" width="0.1524" layer="91"/>
+<wire x1="213.36" y1="91.44" x2="213.36" y2="83.82" width="0.1524" layer="91"/>
 </segment>
 <segment>
@@
 </segment>
 </net>
-<net name="LCD_BIAS_P" class="1">
+<net name="LCD_BIAS_P" class="2">
 <segment>
 <pinref part="LCD" gate="G$1" pin="20"/>
@@
 </segment>
 </net>
-<net name="LCD_BIAS_N" class="0">
+<net name="LCD_BIAS_N" class="2">
 <segment>
 <pinref part="LCD" gate="G$1" pin="19"/>
@@
 </segment>
 </net>
-<net name="VCC256" class="0">
+<net name="VCC256" class="2">
 <segment>
 <pinref part="LCD" gate="G$1" pin="18"/>
@@
 </segment>
 </net>
-<net name="VCC132" class="0">
+<net name="VCC132" class="2">
 <segment>
 <pinref part="LCD" gate="G$1" pin="17"/>
@@
 <net name="LCD_BIASN_SHDN_" class="0">
 <segment>
-<pinref part="U7" gate="G$1" pin="PA5"/>
-<wire x1="236.22" y1="33.02" x2="238.76" y2="33.02" width="0.1524" layer="91"/>
-</segment>
-<segment>
 <pinref part="U6" gate="G$1" pin="SHDN_"/>
 <wire x1="81.28" y1="38.1" x2="73.66" y2="38.1" width="0.1524" layer="91"/>
 </segment>
-</net>
-<net name="LCD_BIASN_DN" class="0">
 <segment>
-<pinref part="U7" gate="G$1" pin="PA6"/>
-<wire x1="236.22" y1="30.48" x2="238.76" y2="30.48" width="0.1524" layer="91"/>
+<pinref part="U7" gate="G$1" pin="PA7"/>
+<wire x1="236.22" y1="27.94" x2="238.76" y2="27.94" width="0.1524" layer="91"/>
 </segment>
+</net>
+<net name="LCD_BIASN_DN" class="0">
 <segment>
 <pinref part="U6" gate="G$1" pin="DN"/>
 <wire x1="81.28" y1="35.56" x2="73.66" y2="35.56" width="0.1524" layer="91"/>
 </segment>
-</net>
-<net name="LCD_BIASN_UP" class="0">
 <segment>
-<pinref part="U7" gate="G$1" pin="PA7"/>
-<wire x1="236.22" y1="27.94" x2="238.76" y2="27.94" width="0.1524" layer="91"/>
+<pinref part="U7" gate="G$1" pin="PA5"/>
+<wire x1="236.22" y1="33.02" x2="238.76" y2="33.02" width="0.1524" layer="91"/>
 </segment>
+</net>
+<net name="LCD_BIASN_UP" class="0">
 <segment>
 <pinref part="U6" gate="G$1" pin="UP"/>
 <wire x1="81.28" y1="33.02" x2="73.66" y2="33.02" width="0.1524" layer="91"/>
 </segment>
-</net>
-<net name="LCD_BIASP_SHDN_" class="0">
 <segment>
-<pinref part="U7" gate="G$1" pin="PA1"/>
-<wire x1="200.66" y1="33.02" x2="198.12" y2="33.02" width="0.1524" layer="91"/>
+<pinref part="U7" gate="G$1" pin="PA6"/>
+<wire x1="236.22" y1="30.48" x2="238.76" y2="30.48" width="0.1524" layer="91"/>
 </segment>
+</net>
+<net name="LCD_BIASP_SHDN_" class="0">
 <segment>
 <pinref part="U5" gate="G$1" pin="SHDN_"/>
 <wire x1="81.28" y1="111.76" x2="73.66" y2="111.76" width="0.1524" layer="91"/>
 </segment>
-</net>
-<net name="LCD_BIASP_DN" class="0">
 <segment>
-<pinref part="U7" gate="G$1" pin="PA2"/>
-<wire x1="200.66" y1="30.48" x2="198.12" y2="30.48" width="0.1524" layer="91"/>
+<pinref part="U7" gate="G$1" pin="PA3"/>
+<wire x1="200.66" y1="27.94" x2="198.12" y2="27.94" width="0.1524" layer="91"/>
 </segment>
+</net>
+<net name="LCD_BIASP_DN" class="0">
 <segment>
 <pinref part="U5" gate="G$1" pin="DN"/>
 <wire x1="81.28" y1="109.22" x2="73.66" y2="109.22" width="0.1524" layer="91"/>
 </segment>
-</net>
-<net name="LCD_BIASP_UP" class="0">
 <segment>
-<pinref part="U7" gate="G$1" pin="PA3"/>
-<wire x1="200.66" y1="27.94" x2="198.12" y2="27.94" width="0.1524" layer="91"/>
+<pinref part="U7" gate="G$1" pin="PA2"/>
+<wire x1="200.66" y1="30.48" x2="198.12" y2="30.48" width="0.1524" layer="91"/>
 </segment>
+</net>
+<net name="LCD_BIASP_UP" class="0">
 <segment>
 <pinref part="U5" gate="G$1" pin="UP"/>
 <wire x1="81.28" y1="106.68" x2="73.66" y2="106.68" width="0.1524" layer="91"/>
 </segment>
+<segment>
+<pinref part="U7" gate="G$1" pin="PA1"/>
+<wire x1="200.66" y1="33.02" x2="198.12" y2="33.02" width="0.1524" layer="91"/>
+</segment>
 </net>
 <net name="N$29" class="0">
@@
 </segment>
 </net>
-<net name="N$17" class="0">
+<net name="LCD_BIAS_P_P1" class="2">
 <segment>
 <pinref part="L2" gate="G$1" pin="2"/>
@@
 </segment>
 </net>
-<net name="N$27" class="0">
+<net name="LCD_BIAS_P_P2" class="2">
 <segment>
 <wire x1="160.02" y1="137.16" x2="160.02" y2="109.22" width="0.1524" layer="91"/>
@@
 </segment>
 </net>
-<net name="N$24" class="0">
+<net name="LCD_BIAS_N_P1" class="2">
 <segment>
 <pinref part="L5" gate="G$1" pin="2"/>
@@
 </segment>
 </net>
-<net name="N$51" class="0">
+<net name="LCD_BIAS_N_P2" class="2">
 <segment>
 <pinref part="C30" gate="C" pin="2"/>

Commit message: add TAPR OHL license
Other:
- note added: "PsiOnSD (c)Greg "GothAck" Miell 2019 Licensed under the TAPR Open Hardware License (www.tapr.org/OHL)"
- note removed: "PsiOnSD (c)Greg "GothAck" Miell 2019"
- moved on the sheet: C14, C17, C18, C19, C20, L4, Q5, Q6, Q7, Q9, R18, R19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

Commit message: Added audio compoments, massive board changes to accommodate physical space & rf restrictions
Parts:
- removed R3: 1k, adafruit:R-US_M0805
- added J1: 0522070433, gothack:0522070433
- added LED2: (no value), adafruit:LEDCHIP-LED0805
- added MK1: SPH0645LM4H-B, gothack:SPH0645LM4H-B
- added SW1: KSM1131, gothack:KSM1131
- added SW2, SW3, SW4: LS12T2-T, gothack:LS12T2-T
- added TP3, TP4, TP5, TP6, TP7: (no value), microbuilder:TESTPOINTROUND1MM
- added U1: USB2514BI-AEZG, USB2514BI-AEZG:USB2514BI-AEZG
- added U9: MAX98357AETE+, MAX98357AETE_:MAX98357AETE+
- added Y2: ABM10-24.000MHZ-E20-T, ABM10-16.000MHZ-D30-T3:ABM10-16.000MHZ-D30-T3
- J2: device 1-2295018-2:1-2295018-2 -> gothack:1-2295018-2
- LED1: device adafruit:LEDCHIPLED_0805 -> adafruit:LEDCHIP-LED0805
- U$1: value LM832 -> LM832EMBEDDED; device LM832:LM832 -> gothack:LM832EMBEDDED
Connections:
- net LCD_BIASN_DN renamed LCD_BIASND_N
- net LCD_BIASP_DN renamed LCD_BIASPD_N
- net U0_CTS renamed UART0_CTS
- net U0_RTS renamed UART0_RTS
- net U0_RXD renamed UART0_RXD
- net U0_TXD renamed UART0_TXD
- net U1_CTS renamed UART1_CTS
- net U1_RTS renamed UART1_RTS
- net U1_RXD renamed UART1_RXD
- net U1_TXD renamed UART1_TXD
- net USBC_DN renamed USBCD_N
- net USBC_DP renamed USBCD_P
- removed net KBD_USB_DN: U3.D-
- removed net KBD_USB_DP: U3.D+
- removed net USB1_DN: U4B.USB1_DM
- removed net USB1_DP: U4B.USB1_DP
- new net AIN0: U4B.AIN0
- new net AIN1: U4B.AIN1
- new net AIN2: U4B.AIN2
- new net AIN3: U4B.AIN3
- new net AIN4: U4B.AIN4
- new net AIN5: U4B.AIN5
- new net AIN6: U4B.AIN6
- new net AIN7: U4B.AIN7
- new net ECAP0_IN_PWM0_OUT: U4C.ECAP0_IN_PWM0_OUT
- new net EMMC_RSTN: U4C.EMMC_RSTN
- new net EMU0: U4B.EMU0
- new net EMU1: U4B.EMU1
- new net GPMC_A0: U4C.GPMC_A0
- new net GPMC_A1: U4C.GPMC_A1
- new net GPMC_A10: U4C.GPMC_A10
- new net GPMC_A11: U4C.GPMC_A11
- new net GPMC_A2: U4C.GPMC_A2
- new net GPMC_A3: U4C.GPMC_A3
- new net GPMC_A4: U4C.GPMC_A4
- new net GPMC_A5: U4C.GPMC_A5
- new net GPMC_A6: U4C.GPMC_A6
- new net GPMC_A7: U4C.GPMC_A7
- new net GPMC_A8: U4C.GPMC_A8
- new net GPMC_A9: U4C.GPMC_A9
- new net GPMC_AD10: U4C.GPMC_AD10
- new net GPMC_AD11: U4C.GPMC_AD11
- new net GPMC_AD12: U4C.GPMC_AD12
- new net GPMC_AD13: U4C.GPMC_AD13
- new net GPMC_AD14: U4C.GPMC_AD14
- new net GPMC_AD15: U4C.GPMC_AD15
- new net GPMC_AD8: U4C.GPMC_AD8
- new net GPMC_AD9: U4C.GPMC_AD9
- new net GPMC_ADVN_ALE: U4C.GPMC_ADVN_ALE
- new net GPMC_BEN0_CLE: U4C.GPMC_BEN0_CLE
- new net GPMC_BEN1: U4C.GPMC_BEN1
- new net GPMC_CLK: U4C.GPMC_CLK
- new net GPMC_CSN0: U4C.GPMC_CSN0
- new net GPMC_CSN3: U4C.GPMC_CSN3
- new net GPMC_OEN_REN: U4C.GPMC_OEN_REN
- new net GPMC_WAIT0: U4C.GPMC_WAIT0
- new net GPMC_WEN: U4C.GPMC_WEN
- new net GPMC_WPN: U4C.GPMC_WPN
- new net KBD_USBD_N: U1.USBDM_DN1/PRT_DIS_M1, U3.D-
- new net KBD_USBD_P: U1.USBDP_DN1/PRT_DIS_P1, U3.D+
- new net MCASP0_ACLKR: MK1.BCLK, U4C.MCASP0_ACLKR
- new net MCASP0_ACLKX: U4C.MCASP0_ACLKX, U9.BCLK
- new net MCASP0_AHCLKR: U4C.MCASP0_AHCLKR
- new net MCASP0_AHCLKX: U4C.MCASP0_AHCLKX
- new net MCASP0_AXR0: U4C.MCASP0_AXR0, U9.DIN
- new net MCASP0_AXR1: MK1.DATA_OUT, U4C.MCASP0_AXR1
- new net MCASP0_FSR: MK1.WS, U4C.MCASP0_FSR
- new net MCASP0_FSX: U4C.MCASP0_FSX, U9.LRCLK
- new net N$15: U1.XTALOUT, Y2.XTAL@2
- new net N$17: TP5.P$1, U4F.VDDS_PLL
- new net N$18: TP6.P$1, U4F.VDD_CORE
- new net N$19: TP7.P$1, U4F.OSC0_TP
- new net N$20: J1.1, J1.2
- new net N$21: U3.UCAP
- new net N$4: U1.XTALIN/CLKIN, Y2.XTAL@1
- new net NC0: U4G.NC@1
- new net NC1: U4G.NC@2
- new net NC10: U4G.NC@11
- new net NC11: U4G.NC@12
- new net NC12: U4G.NC@13
- new net NC13: U4G.NC@14
- new net NC14: U4G.NC@15
- new net NC15: U4G.NC@16
- new net NC16: U4G.NC@17
- new net NC17: U4G.NC@18
- new net NC18: U4G.NC@19
- new net NC19: U4G.NC@20
- new net NC2: U4G.NC@3
- new net NC20: U4G.NC@21
- new net NC21: U4G.NC@22
- new net NC22: U4G.NC@23
- new net NC23: U4G.NC@24
- new net NC24: U4G.NC@25
- new net NC25: U4G.NC@26
- new net NC26: U4G.NC@27
- new net NC27: U4G.NC@28
- new net NC28: U4G.NC@29
- new net NC29: U4G.NC@30
- new net NC3: U4G.NC@4
- new net NC30: U4G.NC@31
- new net NC31: U4G.NC@32
- new net NC32: U4G.NC@33
- new net NC33: U4G.NC@34
- new net NC34: U4G.NC@35
- new net NC35: U4G.NC@36
- new net NC36: U4G.NC@37
- new net NC37: U4G.NC@38
- new net NC38: U4G.NC@39
- new net NC39: U4G.NC@40
- new net NC4: U4G.NC@5
- new net NC40: U4G.NC@41
- new net NC41: U4G.NC@82
- new net NC42: U4G.NC@81
- new net NC43: U4G.NC@80
- new net NC44: U4G.NC@79
- new net NC45: U4G.NC@78
- new net NC46: U4G.NC@77
- new net NC47: U4G.NC@76
- new net NC48: U4G.NC@75
- new net NC49: U4G.NC@74
- new net NC5: U4G.NC@6
- new net NC50: U4G.NC@73
- new net NC51: U4G.NC@72
- new net NC52: U4G.NC@71
- new net NC53: U4G.NC@70
- new net NC54: U4G.NC@69
- new net NC55: U4G.NC@68
- new net NC56: U4G.NC@67
- new net NC57: U4G.NC@66
- new net NC58: U4G.NC@65
- new net NC59: U4G.NC@64
- new net NC6: U4G.NC@7
- new net NC60: U4G.NC@63
- new net NC61: U4G.NC@62
- new net NC62: U4G.NC@61
- new net NC63: U4G.NC@60
- new net NC64: U4G.NC@59
- new net NC65: U4G.NC@58
- new net NC66: U4G.NC@57
- new net NC67: U4G.NC@56
- new net NC68: U4G.NC@55
- new net NC69: U4G.NC@54
- new net NC7: U4G.NC@8
- new net NC70: U4G.NC@53
- new net NC71: U4G.NC@52
- new net NC72: U4G.NC@51
- new net NC73: U4G.NC@50
- new net NC74: U4G.NC@49
- new net NC75: U4G.NC@48
- new net NC76: U4G.NC@47
- new net NC77: U4G.NC@46
- new net NC78: U4G.NC@45
- new net NC79: U4G.NC@44
- new net NC8: U4G.NC@9
- new net NC80: U4G.NC@43
- new net NC81: U4G.NC@42
- new net NC9: U4G.NC@10
- new net OSC0_CTL: U4B.OSC0_CTL
- new net OSC1_GND: U4B.OSC1_GND
- new net OSC1_IN: U4B.OSC1_IN
- new net OSC1_OUT: U4B.OSC1_OUT
- new net PMIC_MUX_IN: U4B.PMIC_MUX_IN
- new net PMIC_MUX_OUT: U4B.PMIC_MUX_OUT
- new net PMIC_NRESET: U4A.PMIC_NRESET
- new net PMIC_TS: U4A.PMIC_TS
- new net PWRONRSTN_OD: U4A.PWRONRSTN_OD
- new net SPI0_CS0: U4C.SPI0_CS0
- new net SPI0_CS1: U4C.SPI0_CS1
- new net SPI0_D0: U4C.SPI0_D0
- new net SPI0_D1: U4C.SPI0_D1
- new net SPI0_SCLK: U4C.SPI0_SCLK
- new net SPKR_LN: J1.3, U9.OUTN
- new net SPKR_LP: J1.4, U9.OUTP
- new net SW_LID: SW1.2, U3.PB7
- new net SW_MEDIA1: SW2.2
- new net SW_MEDIA2: SW3.2
- new net SW_MEDIA3: SW4.2
- new net SYS_ADC_1P8V: U4B.SYS_ADC_1P8V
- new net SYS_VDD1_CTL: U4A.SYS_VDD1_CTL
- new net TCK: U4B.TCK
- new net TDI: U4B.TDI
- new net TDO: U4B.TDO
- new net TMS: U4B.TMS
- new net TRSTN: U4B.TRSTN
- new net USB1D_N: U1.USBDM_UP, U4B.USB1_DM
- new net USB1D_P: U1.USBDP_UP, U4B.USB1_DP
- new net USB1_CE: U4B.USB1_CE
- new net USB1_DRVVBUS: U4B.USB1_DRVVBUS
- new net USB1_VBUS: U4B.USB1_VBUS
- new net USBC_CE: U4B.USB0_CE
- new net USBC_DRVVBUS: U4B.USB0_DRVVBUS
- new net USB_DN2D_N: U1.USBDM_DN2/PRT_DIS_M2
- new net USB_DN2D_P: U1.USBDP_DN2/PRT_DIS_P2
- new net USB_DN3D_N: U1.USBDM_DN3/PRT_DIS_M3
- new net USB_DN3D_P: U1.USBDP_DN3/PRT_DIS_P3
- new net USB_DN4D_N: U1.USBDM_DN4/PRT_DIS_M4
- new net USB_DN4D_P: U1.USBDP_DN4/PRT_DIS_P4
- new net VDDS_RTC@2: U4A.VDDS_RTC@2
- new net VREFN: U4B.VREFN
- new net VREFP: U4B.VREFP
- new net WARMRSTN: U4A.WARMRSTN
- new net XDMA_EVENT_INTR0: U4C.XDMA_EVENT_INTR0
- new net XDMA_EVENT_INTR1: U4C.XDMA_EVENT_INTR1
- net +3V3: now also MK1.VDD, U1.VDD33_1, U1.VDD33_2, U1.VDDA33_1, U1.VDDA33_2, U1.VDDA33_3, U1.VDDA33_4, U9.VDD
- net GND: now also MK1.GND, SW1.1, SW2.1, SW3.1, SW4.1, U1.PWRPAD, U4B.AGND_ADC, U9.GND, Y2.2, Y2.4; no longer R3.2
- net I2C0_SCL: now also U1.SCL/SMBCLK/CFG_SEL0
- net I2C0_SDA: now also U1.SDA/SMBDATA/NON_REM1
- net KBDAVR_VCC: no longer U3.UCAP
- net N$2: now also TP3.P$1, U4F.VDD_MPU; no longer LED1.C, R3.1
- net N$6: now also TP4.P$1, U4F.VDDS_DDR; no longer LED1.A, U3.PB7
- net USBC_ID: now also U4B.USB0_ID
Other:
- note added: "Power"
- note added: "SD, WiFi, LCD"
- note added: "SiP Ground / Misc"
- note added: "This sheet intentionally left blank"
- note added: "USB, Audio, Keyboard"
- note removed: "KBD / SiP MISC"
- note removed: "USB / WIFI / SD"
